File: joost.kicad_blocks/rp2354.kicad_block/rp2354.kicad_sch (KiCad schematic)
At the start: 48 parts, among them U10 GT-USB-7010ASV, U12 W25Q128, U2 RP2350_80QFN, U32 APS6404L-3SQR-SN_C5333729, Y1 ABM8-272-T3

Commit message: -
Parts:
- removed R154, R155, R156, R157: 1kΩ, PCM_JLCPCB:R_0402, symbol PCM_JLCPCB-Resistors:0402,1kΩ
- L1: footprint easyeda2kicad:IND-SMD_L2.0-W1.6_AOTA-B201610S3R3-101-T -> joost:IND-SMD_L2.0-W1.6_AOTA-B201610S3R3-101-T; symbol easyeda2kicad:AOTA-B201610S3R3-101-T -> joost:AOTA-B201610S3R3-101-T; MPN (none) -> AOTA-B201610S3R3-101-T; Manufacturer (none) -> ABRACON
- S1: renamed from S2; footprint PCM_JLCPCB:SW-SMD_4P-L5.1-W5.1-P3.70-LS6.5-TL-2 -> joost:joost SW-SMD_4P-L5.1-W5.1-P3.70-LS6.5-TL_H1.5; symbol PCM_JLCPCB-Connectors_Buttons:Tactile Button, 160gf, 12V, 50mA, 5.1mm -> joost:SW_SPST; Actuator Style Round Button -> (none); Actuator/Cap Color Golden -> (none); Attrition Qty 5 -> (none); Category Switches,Tactile Switches -> (none); Circuit SPST -> (none); Class Basic Component -> (none); Contact Current 50mA -> (none); Manufacturer XKB Connectivity -> (none); Mechanical Life 100000 Times -> (none); Minimum Qty 10 -> (none); Mounting Style Brick nogging -> (none); Operating Force 160gf -> (none); Operating Temperature -30°C~+85°C -> (none); Part TS-1187A-B-A-B -> (none); Price 0.025USD -> (none); Process SMT -> (none); Stock 472664 -> (none); Strike Gundam NO -> (none); Switch Height 1.5mm -> (none); Switch Length 5.1mm -> (none); Switch Width 5.1mm -> (none); Voltage Rating (Dc) 12V -> (none); With Lamp No -> (none)
- S2: renamed from S1; footprint PCM_JLCPCB:SW-SMD_4P-L5.1-W5.1-P3.70-LS6.5-TL-2 -> joost:joost SW-SMD_4P-L5.1-W5.1-P3.70-LS6.5-TL_H1.5; symbol PCM_JLCPCB-Connectors_Buttons:Tactile Button, 160gf, 12V, 50mA, 5.1mm -> joost:SW_SPST; Actuator Style Round Button -> (none); Actuator/Cap Color Golden -> (none); Attrition Qty 5 -> (none); Category Switches,Tactile Switches -> (none); Circuit SPST -> (none); Class Basic Component -> (none); Contact Current 50mA -> (none); Manufacturer XKB Connectivity -> (none); Mechanical Life 100000 Times -> (none); Minimum Qty 10 -> (none); Mounting Style Brick nogging -> (none); Operating Force 160gf -> (none); Operating Temperature -30°C~+85°C -> (none); Part TS-1187A-B-A-B -> (none); Price 0.025USD -> (none); Process SMT -> (none); Stock 472664 -> (none); Strike Gundam NO -> (none); Switch Height 1.5mm -> (none); Switch Length 5.1mm -> (none); Switch Width 5.1mm -> (none); Voltage Rating (Dc) 12V -> (none); With Lamp No -> (none)
- U1: renamed from U10; footprint easyeda2kicad:USB-C-SMD_G-SWITCH_GT-USB-7010ASV -> joost:USB-C-SMD_G-SWITCH_GT-USB-7010ASV; symbol easyeda2kicad:GT-USB-7010ASV -> joost:GT-USB-7010ASV
- renumbered C38 to C1, C16 to C10, C17 to C11, C18 to C12, C20 to C13, C39 to C14, C21 to C15, C36 to C16, C19 to C17, C3 to C18, C12 to C19, C7 to C2, C10 to C20, C4 to C3, C6 to C4, C9 to C5, C8 to C6, C13 to C7, C14 to C8, C15 to C9, R167 to R1, R3 to R10, R7 to R11, R150 to R12, R151 to R13, R2 to R14, R42 to R15, R46 to R16, R44 to R17, R43 to R18, R45 to R19, R166 to R2, R8 to R20, R15 to R3, R10 to R4, R4 to R5, U12 to U3, U32 to U4
Connections:
- net GND: now also S1.1 (A); no longer S1.4 (D)
- net ~{USB_BOOT}: now also S1.2 (B); no longer S1.1 (A)
- net at S2.2 (B): now also U2.35 (RUN)
- net A0: no longer names the net of U2.11 (GPIO12)
- net A1: no longer names the net of U2.12 (GPIO13)
- net A2: no longer names the net of U2.13 (GPIO14)
- net ADC0: no longer names the net of U2.49 (GPIO40_ADC0)
- net ADC1: no longer names the net of U2.52 (GPIO41_ADC1)
- net ADC2: no longer names the net of U2.53 (GPIO42_ADC2)
- net ADC3: no longer names the net of U2.54 (GPIO43_ADC3)
- net GPIO24: no longer names the net of U2.25 (GPIO24)
- net GPIO25: no longer names the net of U2.26 (GPIO25)
- net GPIO26: no longer names the net of U2.27 (GPIO26)
- net GPIO27: no longer names the net of U2.28 (GPIO27)
- net GPIO28: no longer names the net of U2.36 (GPIO28)
- net GPIO29: no longer names the net of U2.37 (GPIO29)
- net GPIO30: no longer names the net of U2.38 (GPIO30)
- net GPIO31: no longer names the net of U2.39 (GPIO31)
- net GPIO34: no longer names the net of U2.43 (GPIO34)
- net GPIO35: no longer names the net of U2.44 (GPIO35)
- net GPIO38: no longer names the net of U2.47 (GPIO38)
- net GPIO39: no longer names the net of U2.48 (GPIO39)
- net GPIO45: no longer names the net of U2.56 (GPIO45_ADC5)
- net GPIO46: no longer names the net of U2.57 (GPIO46_ADC6)
- net LEDBANK0_EN: no longer names the net of U2.1 (GPIO4)
- net LEDBANK1_EN: no longer names the net of U2.2 (GPIO5)
- net LEDBANK2_EN: no longer names the net of U2.3 (GPIO6)
- net LEDBANK3_EN: no longer names the net of U2.4 (GPIO7)
- net MASTER_AUX1: no longer names the net of U2.20 (GPIO20)
- net MASTER_AUX2: no longer names the net of U2.21 (GPIO21)
- net MAX_DE: no longer names the net of U2.45 (GPIO36)
- net SCL: no longer names the net of U2.80 (GPIO3)
- net SDA: no longer names the net of U2.79 (GPIO2)
- net SLAVE_AUX1: no longer names the net of U2.22 (GPIO22)
- net SLAVE_AUX2: no longer names the net of U2.23 (GPIO23)
- net SPI_MASTER_CSn: no longer names the net of U2.17 (GPIO17)
- net SPI_MASTER_MISO: no longer names the net of U2.16 (GPIO16)
- net SPI_MASTER_MOSI: no longer names the net of U2.19 (GPIO19)
- net SPI_MASTER_SCK: no longer names the net of U2.18 (GPIO18)
- net UART_RX: no longer names the net of U2.42 (GPIO33)
- net UART_TX: no longer names the net of U2.40 (GPIO32)
- net USERBTN: no longer names the net of U2.78 (GPIO1)
- net USERLED: no longer names the net of U2.14 (GPIO15)
- net V5SENSE: no longer names the net of U2.55 (GPIO44_ADC4)
- no-connect marks 7 -> 2
Other:
- moved on the sheet: R3
